Commit message: create launch file

File: src/explorer_bot/urdf/fast.urdf (robot description, URDF)
Before this commit: robot dolly, 5 links, 4 joints
Links:
- removed link base
- removed link world
- added link base_footprint, mass 1; collision box size=0.75 0.4 0.1; visual box size=0.75 0.4 0.1
- added link laser, mass 1; collision sphere radius=.08; visual cylinder length=0.05 radius=0.05
Joints:
- removed joint base_joint
- added joint laser_joint: type fixed, parent base_footprint, child laser, origin xyz=-0.32 0.0 0.08 rpy=0.0 0.0 3.14, axis 0 0 1

File: src/explorer_bot/urdf/shape.urdf (robot description, URDF)
Before this commit: robot multipleshapes, 2 links, 1 joints
Links:
- removed link right_leg
- added link front_caster_of_wheel, mass 0.1; collision box size=0.1 0.1 0.1; visual box size=0.1 0.1 0.1
- added link front_wheel, mass 0.1; collision cylinder length=0.05 radius=0.035; visual cylinder length=0.05 radius=0.035
- added link laser_scanner, mass 1e-5; collision box size=0.1 0.1 0.1; visual box size=0.1 0.1 0.1
- added link left_wheel, mass 0.1; collision cylinder length=0.05 radius=0.035; visual cylinder length=0.05 radius=0.035
- added link right_wheel, mass 0.1; collision cylinder length=0.05 radius=0.035; visual cylinder length=0.05 radius=0.035
- link base_link: mass None -> 1.0; geometry collision box size=0.6 0.3 0.1; visual box size=0.6 0.3 0.1
Joints:
- removed joint base_to_right_leg
- added joint front_caster_of_wheel_joint: type continuous, parent base_link, child front_caster_of_wheel, origin xyz=0.3 0.0 0.0 rpy=0.0 0.0 0.0, axis 0.0 0.0 1
- added joint front_wheel_joint: type continuous, parent front_caster_of_wheel, child front_wheel, origin xyz=0.05 0.0 -0.05 rpy=-1.5708 0.0 0.0, axis 0.0 0.0 1
- added joint laser_scanner_joint: type fixed, parent base_link, child laser_scanner, origin xyz=0.0 0.0 0.08 rpy=0.0 0.0 0.0, axis 0.0 1 0.0
- added joint left_wheel_joint: type continuous, parent base_link, child left_wheel, origin xyz=-0.2825 0.125 -0.05 rpy=-1.5708 0.0 0.0, axis 0.0 0.0 1
- added joint right_wheel_joint: type continuous, parent base_link, child right_wheel, origin xyz=-0.2825 -0.125 -0.05 rpy=-1.5708 0.0 0.0, axis 0.0 0.0 1
